File: DroneMotor.kicad_pcb (KiCad board)
At the start: 2 copper layers, 184 x 184 mm, 49 parts, among them Q1 ISCH54N04NM7V, Q10 ISCH54N04NM7V, Q11 ISCH54N04NM7V, Q12 ISCH54N04NM7V, Q13 ISCH54N04NM7V, Q14 ISCH54N04NM7V, Q15 ISCH54N04NM7V, Q16 ISCH54N04NM7V, Q17 ISCH54N04NM7V, Q18 ISCH54N04NM7V, Q19 ISCH54N04NM7V, Q2 ISCH54N04NM7V, Q20 ISCH54N04NM7V, Q21 ISCH54N04NM7V, Q22 ISCH54N04NM7V, Q23 ISCH54N04NM7V, Q24 ISCH54N04NM7V, Q3 ISCH54N04NM7V, Q4 ISCH54N04NM7V, Q5 ISCH54N04NM7V, Q6 ISCH54N04NM7V, Q7 ISCH54N04NM7V, Q8 ISCH54N04NM7V, Q9 ISCH54N04NM7V, U1 MKV58F1M0VLQ22, U10 UCC27211DRMR, U11 UCC27211DRMR, U12 UCC27211DRMR, U13 UCC27211DRMR, U2 UCC27211DRMR, U3 UCC27211DRMR, U4 UCC27211DRMR, U5 UCC27211DRMR, U6 UCC27211DRMR, U7 UCC27211DRMR, U8 UCC27211DRMR, U9 UCC27211DRMR

Commit message: add
Parts:
- removed U10, U11, U12, U13, U3, U4, U5, U6, U7, U8, U9: UCC27211DRMR, footprints:VSON-8_L4.0-W4.0-P0.80-TL-EP
- TP11, TP2, TP5, TP8: value HSB -> HSA
- TP12, TP3, TP6, TP9: value HSC -> HSA
- moved Q7 151.6 mm to (143.8, 157.3), turned to 90 degrees
- moved Q11 150.7 mm to (143.8, 130.7), turned to 90 degrees
- moved Q9 150.6 mm to (144.3, 143.5), turned to 90 degrees
- moved TP5 150.3 mm to (132.9, 140.8), turned to 90 degrees
- moved TP4 150.1 mm to (133.0, 153.7), turned to 90 degrees
- moved TP6 149.0 mm to (133.0, 128.0), turned to 90 degrees
- moved Q8 130.6 mm to (143.8, 150.7), turned to 90 degrees
- moved Q10 130.3 mm to (144.3, 136.9), turned to 90 degrees
- moved Q12 129.5 mm to (143.8, 124.1), turned to 90 degrees
- moved TP7 128.0 mm to (302.4, 126.9), turned to 0 degrees
- moved TP1 126.7 mm to (214.6, 233.0)
- moved Q1 123.6 mm to (212.4, 224.5), turned to 0 degrees
- moved TP3 122.8 mm to (232.3, 234.0)
- moved Q14 121.4 mm to (288.6, 129.4), turned to -90 degrees
- moved Q5 121.3 mm to (229.0, 226.0), turned to 0 degrees
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Connections:
- Q1 pad 1: Net-(Q1-S-Pad1) -> Net-(U2-HS)
- Q1 pad 2: Net-(Q1-S-Pad1) -> Net-(U2-HS)
- Q1 pad 3: Net-(Q1-S-Pad1) -> Net-(U2-HS)
- Q1 pad 5: Net-(Q1-D-Pad5) -> VCC_DC+
- Q1 pad 6: Net-(Q1-D-Pad5) -> VCC_DC+
- Q1 pad 7: Net-(Q1-D-Pad5) -> VCC_DC+
- Q1 pad 8: Net-(Q1-D-Pad5) -> VCC_DC+
- Q11 pad 5: Net-(Q11-D-Pad5) -> VCC_DC+
- Q11 pad 6: Net-(Q11-D-Pad5) -> VCC_DC+
- Q11 pad 7: Net-(Q11-D-Pad5) -> VCC_DC+
- Q11 pad 8: Net-(Q11-D-Pad5) -> VCC_DC+
- Q12 pad 1: Net-(Q12-S-Pad1) -> Net-(Q10-S-Pad1)
- Q12 pad 2: Net-(Q12-S-Pad1) -> Net-(Q10-S-Pad1)
- Q12 pad 3: Net-(Q12-S-Pad1) -> Net-(Q10-S-Pad1)
- Q13 pad 5: Net-(Q13-D-Pad5) -> VCC_DC+
- Q13 pad 6: Net-(Q13-D-Pad5) -> VCC_DC+
- Q13 pad 7: Net-(Q13-D-Pad5) -> VCC_DC+
- Q13 pad 8: Net-(Q13-D-Pad5) -> VCC_DC+
- Q15 pad 5: Net-(Q13-D-Pad5) -> VCC_DC+
- Q15 pad 6: Net-(Q13-D-Pad5) -> VCC_DC+
- Q15 pad 7: Net-(Q13-D-Pad5) -> VCC_DC+
- Q15 pad 8: Net-(Q13-D-Pad5) -> VCC_DC+
- Q16 pad 1: Net-(Q16-S-Pad1) -> Net-(Q14-S-Pad1)
- Q16 pad 2: Net-(Q16-S-Pad1) -> Net-(Q14-S-Pad1)
- Q16 pad 3: Net-(Q16-S-Pad1) -> Net-(Q14-S-Pad1)
- Q17 pad 5: Net-(Q13-D-Pad5) -> VCC_DC+
- Q17 pad 6: Net-(Q13-D-Pad5) -> VCC_DC+
- Q17 pad 7: Net-(Q13-D-Pad5) -> VCC_DC+
- Q17 pad 8: Net-(Q13-D-Pad5) -> VCC_DC+
- Q18 pad 1: Net-(Q18-S-Pad1) -> Net-(Q14-S-Pad1)
- Q18 pad 2: Net-(Q18-S-Pad1) -> Net-(Q14-S-Pad1)
- Q18 pad 3: Net-(Q18-S-Pad1) -> Net-(Q14-S-Pad1)
- Q19 pad 5: Net-(Q19-D-Pad5) -> VCC_DC+
- Q19 pad 6: Net-(Q19-D-Pad5) -> VCC_DC+
- Q19 pad 7: Net-(Q19-D-Pad5) -> VCC_DC+
- Q19 pad 8: Net-(Q19-D-Pad5) -> VCC_DC+
- Q2 pad 5: Net-(Q1-S-Pad1) -> Net-(U2-HS)
- Q2 pad 6: Net-(Q1-S-Pad1) -> Net-(U2-HS)
- Q2 pad 7: Net-(Q1-S-Pad1) -> Net-(U2-HS)
- Q2 pad 8: Net-(Q1-S-Pad1) -> Net-(U2-HS)
- Q21 pad 5: Net-(Q19-D-Pad5) -> VCC_DC+
- Q21 pad 6: Net-(Q19-D-Pad5) -> VCC_DC+
- Q21 pad 7: Net-(Q19-D-Pad5) -> VCC_DC+
- Q21 pad 8: Net-(Q19-D-Pad5) -> VCC_DC+
- Q22 pad 1: Net-(Q22-S-Pad1) -> Net-(Q20-S-Pad1)
- Q22 pad 2: Net-(Q22-S-Pad1) -> Net-(Q20-S-Pad1)
- Q22 pad 3: Net-(Q22-S-Pad1) -> Net-(Q20-S-Pad1)
- Q23 pad 5: Net-(Q19-D-Pad5) -> VCC_DC+
- Q23 pad 6: Net-(Q19-D-Pad5) -> VCC_DC+
- Q23 pad 7: Net-(Q19-D-Pad5) -> VCC_DC+
- Q23 pad 8: Net-(Q19-D-Pad5) -> VCC_DC+
- Q24 pad 1: Net-(Q24-S-Pad1) -> Net-(Q20-S-Pad1)
- Q24 pad 2: Net-(Q24-S-Pad1) -> Net-(Q20-S-Pad1)
- Q24 pad 3: Net-(Q24-S-Pad1) -> Net-(Q20-S-Pad1)
- Q3 pad 5: Net-(Q1-D-Pad5) -> VCC_DC+
- Q3 pad 6: Net-(Q1-D-Pad5) -> VCC_DC+
- Q3 pad 7: Net-(Q1-D-Pad5) -> VCC_DC+
- Q3 pad 8: Net-(Q1-D-Pad5) -> VCC_DC+
- Q4 pad 1: Net-(Q4-S-Pad1) -> Net-(Q2-S-Pad1)
- Q4 pad 2: Net-(Q4-S-Pad1) -> Net-(Q2-S-Pad1)
- Q4 pad 3: Net-(Q4-S-Pad1) -> Net-(Q2-S-Pad1)
- Q5 pad 5: Net-(Q1-D-Pad5) -> VCC_DC+
- Q5 pad 6: Net-(Q1-D-Pad5) -> VCC_DC+
- Q5 pad 7: Net-(Q1-D-Pad5) -> VCC_DC+
- Q5 pad 8: Net-(Q1-D-Pad5) -> VCC_DC+
- Q6 pad 1: Net-(Q6-S-Pad1) -> Net-(Q2-S-Pad1)
- Q6 pad 2: Net-(Q6-S-Pad1) -> Net-(Q2-S-Pad1)
- Q6 pad 3: Net-(Q6-S-Pad1) -> Net-(Q2-S-Pad1)
- Q7 pad 5: Net-(Q11-D-Pad5) -> VCC_DC+
- Q7 pad 6: Net-(Q11-D-Pad5) -> VCC_DC+
- Q7 pad 7: Net-(Q11-D-Pad5) -> VCC_DC+
- Q7 pad 8: Net-(Q11-D-Pad5) -> VCC_DC+
- Q8 pad 1: Net-(Q8-S-Pad1) -> Net-(Q10-S-Pad1)
- Q8 pad 2: Net-(Q8-S-Pad1) -> Net-(Q10-S-Pad1)
- Q8 pad 3: Net-(Q8-S-Pad1) -> Net-(Q10-S-Pad1)
- Q9 pad 5: Net-(Q11-D-Pad5) -> VCC_DC+
- Q9 pad 6: Net-(Q11-D-Pad5) -> VCC_DC+
- Q9 pad 7: Net-(Q11-D-Pad5) -> VCC_DC+
- Q9 pad 8: Net-(Q11-D-Pad5) -> VCC_DC+
- TP1 pad 1: Net-(Q1-S-Pad1) -> Net-(U2-HS)
- U2 pad 1: unconnected-(U2-VDD-Pad1) -> VCC
- U2 pad 2: unconnected-(U2-HB-Pad2) -> Net-(U2-HB)
- U2 pad 3: unconnected-(U2-HO-Pad3) -> Net-(U2-HO)
- U2 pad 4: unconnected-(U2-HS-Pad4) -> Net-(U2-HS)
- U2 pad 5: unconnected-(U2-HI-Pad5) -> /motor1/PWM_A_HS
- U2 pad 6: unconnected-(U2-LI-Pad6) -> /motor1/PWM_A_LS
- U2 pad 7: unconnected-(U2-VSS-Pad7) -> GNDREF
- U2 pad 8: unconnected-(U2-LO-Pad8) -> Net-(U2-LO)
- U2 pad 9: unconnected-(U2-PAD-Pad9) -> GNDREF
