File: DroneMotor.kicad_sch (KiCad schematic)
At the start: 0 parts

Commit message: add rev
Other:
- added sheet Controller (controller.kicad_sch)
- added sheet motor1 (motor1.kicad_sch)
- added sheet motor2 (motor2.kicad_sch)
- added sheet motor3 (motor3.kicad_sch)
- added sheet motor4 (motor4.kicad_sch)

Commit message: add ti version
Other:
- added sheet controllerConfig (controllerConfig.kicad_sch)
- added sheet controllerpower (controllerpower.kicad_sch)
- sheet Controller ports: added M1_I_SENSE_C, M1_PWM_B_LS, M1_PWM_C_HS, M1_PWM_C_LS, M1_SS, M1_V_SENSE_DCBUS, M2_BEMF_A, M2_BEMF_B, M2_BEMF_C, M2_DRV_INT, M2_DRV_OS, M2_INPUT, M2_I_DCB, M2_I_SENSE_C, M2_LED_1, M2_PWM_A_HS, M2_PWM_A_LS, M2_PWM_B_HS, M2_PWM_B_LS, M2_PWM_C_HS, M2_PWM_C_LS, M2_SS, M2_V_SENSE_DCBUS, M3_BEMF_A, M3_BEMF_B, M3_BEMF_C, M3_DRV_INT, M3_DRV_OC, M3_INPUT, M3_I_DCB, M3_I_SENSE_C, M3_LED_1, M3_PWM_A_HS, M3_PWM_A_LS, M3_PWM_B_HS, M3_PWM_B_LS, M3_PWM_C_HS, M3_PWM_C_LS, M3_SS, M3_V_SENSE_DCBUS, M4_BEMF_A, M4_BEMF_B, M4_BEMF_C, M4_DRV_INT, M4_DRV_OC, M4_INPUT, M4_I_DCB, M4_I_SENSE_C, M4_LED_1, M4_PWM_A_HS, M4_PWM_A_LS, M4_PWM_B_HS, M4_PWM_B_LS, M4_PWM_C_HS, M4_PWM_C_LS, M4_SS, M4_V_SENSE_DCBUS, MISO, MOSI, RESET_MCU, SCLK, SWDCLK, SWDIO, SWO, UART_RX, UART_TX, U_DCB; removed none
- sheet motor1 ports: added BEMF_A, BEMF_B, BEMF_C, I_SENSE_C, PWM_A_HS, PWM_A_LS, PWM_B_HS, PWM_B_LS, PWM_C_HS, PWM_C_LS, V_SENSE_DCBUS; removed none
- sheet motor2 ports: added BEMF_A, BEMF_B, BEMF_C, I_SENSE_C, PWM_A_HS, PWM_A_LS, PWM_B_HS, PWM_B_LS, PWM_C_HS, PWM_C_LS, V_SENSE_DCBUS; removed none
- sheet motor3 ports: added BEMF_A, BEMF_B, BEMF_C, I_SENSE_C, PWM_A_HS, PWM_A_LS, PWM_B_HS, PWM_B_LS, PWM_C_HS, PWM_C_LS, V_SENSE_DCBUS; removed none
- sheet motor4 ports: added BEMF_A, BEMF_B, BEMF_C, I_SENSE_C, PWM_A_HS, PWM_A_LS, PWM_B_HS, PWM_B_LS, PWM_C_HS, PWM_C_LS, V_SENSE_DCBUS; removed none
