File: controller.kicad_sch (KiCad schematic)
At the start: 30 parts, among them U1 MKV58F1M0VLQ22, Y1 8MHZ

Commit message: add ti version
Parts:
- removed C1, C13, C14: 2.2uF, symbol Device:C_US
- removed C10, C11, C12, C2, C3, C4, C5, C6, C7, C8, C9: 0.1uF, symbol Device:C_US
- removed C15, C16: 22pF, symbol Device:C
- removed D1, D2, D3, D4, D5: D_Schottky, symbol Device:D_Schottky
- removed R1, R2: 2.2K, symbol Device:R_US
- removed R3: 1K, symbol Device:R_US
- removed R4, R5: 7.5K, symbol Device:R_US
- removed R6, R7: 10K, symbol Device:R_US
- removed U1: MKV58F1M0VLQ22, footprints:LQFP144_SOT486-2_NXP, symbol AzizFaozi:MKV58F1M0VLQ22
- removed Y1: 8MHZ, symbol Device:Crystal_GND24
- added U1: XF28388DPTPS, footprints:PTP0176F-IPC_A, symbol TMS320F28388D:XF28388DPTPS
Connections:
- net M1_PWM_A_HS: now also U1.161 (GPIO1)
- net M1_PWM_A_LS: now also U1.160 (GPIO0)
- net M1_PWM_B_HS: now also U1.163 (GPIO3)
- net M1_PWM_B_LS: now also U1.162 (GPIO2)
- net M1_PWM_C_HS: now also U1.165 (GPIO5)
- net M1_PWM_C_LS: now also U1.164 (GPIO4)
- net M2_PWM_A_HS: now also U1.167 (GPIO7)
- net M2_PWM_A_LS: now also U1.166 (GPIO6)
- net M2_PWM_B_HS: now also U1.19 (GPIO9)
- net M2_PWM_B_LS: now also U1.18 (GPIO8)
- net M2_PWM_C_HS: now also U1.2 (GPIO11)
- net M2_PWM_C_LS: now also U1.1 (GPIO10)
- net M3_PWM_A_HS: now also U1.5 (GPIO13)
- net M3_PWM_A_LS: now also U1.4 (GPIO12)
- net M3_PWM_B_HS: now also U1.7 (GPIO15)
- net M3_PWM_B_LS: now also U1.6 (GPIO14)
- net M3_PWM_C_HS: now also U1.9 (GPIO17)
- net M3_PWM_C_LS: now also U1.8 (GPIO16)
- net M4_PWM_A_HS: now also U1.10 (GPIO18)
- net M4_PWM_A_LS: now also U1.12 (GPIO19)
- net M4_PWM_B_HS: now also U1.13 (GPIO20)
- net M4_PWM_B_LS: now also U1.14 (GPIO21)
- net M4_PWM_C_HS: now also U1.22 (GPIO22)
- net M4_PWM_C_LS: now also U1.23 (GPIO23)
- new net EPWM13A: U1.24 (GPIO24)
- new net EPWM13B: U1.25 (GPIO25)
- new net EPWM14A: U1.27 (GPIO26)
- new net EPWM14B: U1.28 (GPIO27)
- new net EPWM15A: U1.64 (GPIO28)
- new net EPWM15B: U1.65 (GPIO29)
- new net EPWM16A: U1.63 (GPIO30)
- new net EPWM16B: U1.66 (GPIO31)
- new net I2CA_SCL: U1.69 (GPIO33)
- new net I2CA_SDA: U1.67 (GPIO32)
- no-connect marks 40 -> 0
Other:
- added sheet controllerADC (controllerADC.kicad_sch)
