File: motor1.kicad_sch (KiCad schematic)
At the start: 30 parts, among them Q1 ISCH54N04NM7V, Q2 ISCH54N04NM7V, Q3 ISCH54N04NM7V, Q4 ISCH54N04NM7V, Q5 ISCH54N04NM7V, Q6 ISCH54N04NM7V, U2 UCC27211DRMR, U6 UCC27211DRMR, U7 UCC27211DRMR

Commit message: add ti version
Parts:
- removed C18: 390pF, symbol Device:C_US
- removed R10, R13, R14, R15, R16: 22, symbol Device:R_US
- removed R19: 4.70K, symbol Device:R_US
- removed U6, U7: UCC27211DRMR, footprints:VSON-8_L4.0-W4.0-P0.80-TL-EP, symbol droneUltimate:UCC27211DRMR
- added C12, C138, C15, C16, C24: 2.2uF, Capacitor_SMD:C_0402_1005Metric, symbol Device:C_US
- added C22, C23, C32: 0.1uF, Capacitor_SMD:C_0603_1608Metric, symbol Device:C
- added C26, C27, C28, C34: 0.1uF, Capacitor_SMD:C_0402_1005Metric, symbol Device:C_US
- added R23, R25, R31: 18K, Resistor_SMD:R_0603_1608Metric, symbol Device:R_US
- added R24, R30: 68K, Resistor_SMD:R_0603_1608Metric, symbol Device:R_US
- added R3: 330, Resistor_SMD:R_0402_1005Metric, symbol Device:R_US
- added R32, R5, R6, R7: 10, Resistor_SMD:R_0603_1608Metric, symbol Device:R_US
- added R33: 1K, Resistor_SMD:R_0603_1608Metric, symbol Device:R_US
- added R42: 0.002, Resistor_SMD:R_2512_6332Metric, symbol Device:R_US
- added U3, U5: UCC27211DRMR, footprints:VSON-8_L4.0-W4.0-P0.80-TL-EP, symbol droneUltimate:UCC27211DRMR
- added U4: OPA4374AIPWR, footprints:PW14, symbol droneUltimate:OPA4374AIPWR
- C17: value 390pF -> 0.1uF; footprint (none) -> Capacitor_SMD:C_0402_1005Metric; lcsc_id (none) -> C60474; price (none) -> 0.001
- C19: value 390pF -> 2.2uF; footprint (none) -> Capacitor_SMD:C_0402_1005Metric; Voltage Rating (none) -> 25V; lcsc_id (none) -> C6119765; price (none) -> 0.0079
- R11, R8: value 22 -> 10; footprint (none) -> Resistor_SMD:R_0603_1608Metric; lcsc_id (none) -> C136596; price (none) -> 0.0015
- R12: value 22 -> 33K; footprint (none) -> Resistor_SMD:R_0603_1608Metric; lcsc_id (none) -> C2907028; price (none) -> 0.0011
- R17: value 4.70K -> 1K; footprint (none) -> Resistor_SMD:R_0603_1608Metric; lcsc_id (none) -> C2907002; price (none) -> 0.0012
- R18: value 1K -> 33K; footprint (none) -> Resistor_SMD:R_0603_1608Metric; lcsc_id (none) -> C2907028; price (none) -> 0.0011
- R20, R22: value 1K -> 68K; footprint (none) -> Resistor_SMD:R_0603_1608Metric; lcsc_id (none) -> C705793; price (none) -> 0.0257
- R21: value 4.70K -> 18K; footprint (none) -> Resistor_SMD:R_0603_1608Metric; lcsc_id (none) -> C309650; price (none) -> 0.0265
- R9: value 22 -> 330; footprint (none) -> Resistor_SMD:R_0402_1005Metric; lcsc_id (none) -> C105875; price (none) -> 0.0008
Connections:
- net BEMF_A: now also R20.2, R21.1, C26.1; no longer C19.1, R21.2, R22.1
- net BEMF_B: now also R22.2, C27.1, R23.1; no longer R20.1
- net BEMF_C: now also C34.1, R30.2, R31.1; no longer C17.1, R17.2, R18.1
- net GNDD: now also R17.1, R21.2, C12.2, C15.2, C24.2, C26.2, C27.2, C28.2, C34.2, R23.2, R25.2, R3.1, R31.2, R42.2, U4.11 (V-); no longer C19.2, R18.2, R20.2, R22.2
- net PA_HS_S: now also Q1.1 (S), Q1.2 (S), Q1.3 (S), Q2.5 (D), Q2.6 (D), Q2.7 (D), Q2.8 (D), R20.1, TP1.1, U2.4 (HS), C22.2; no longer R21.1
- net PB_HS_S: now also Q3.1 (S), Q3.2 (S), Q3.3 (S), Q4.5 (D), Q4.6 (D), Q4.7 (D), Q4.8 (D), R22.1, TP2.1, C23.2, U3.4 (HS)
- net PC_HS_S: now also Q5.1 (S), Q5.2 (S), Q5.3 (S), Q6.5 (D), Q6.6 (D), Q6.7 (D), Q6.8 (D), TP3.1, C32.2, R30.1, U5.4 (HS); no longer R17.1
- net at R11.2: now also Q5.4 (G); no longer Q3.4 (G)
- net VCC_DC+: now reaches Q1.5 (D), Q1.6 (D), Q1.7 (D), Q1.8 (D), Q3.5 (D), Q3.6 (D), Q3.7 (D), Q3.8 (D), Q5.5 (D), Q5.6 (D), Q5.7 (D), Q5.8 (D)
- net VCC_DC+: now also C12.1, C15.1, C24.1, R24.1
- net at Q1.4 (G): now also R6.2; no longer R8.2
- net at R12.1: now also R33.2, U4.6 (-)
- net at Q4.4 (G): now also R8.2; no longer R12.2
- net VCC_12V: now reaches U2.1 (VDD)
- net VCC_12V: now also C19.1, C138.1, C16.1, U3.1 (VDD), U5.1 (VDD)
- net at U2.2 (HB): now also C22.1
- net at U2.3 (HO): now also R6.1
- net PWM_A_HS: now reaches U2.5 (HI)
- net PWM_A_LS: now reaches U2.6 (LI)
- net GNDREF: now reaches U2.7 (VSS)
- net GNDREF: now also C19.2, U2.9 (PAD), C138.2, C16.2, U3.7 (VSS), U3.9 (PAD), U5.7 (VSS), U5.9 (PAD)
- net at U2.8 (LO): now also R5.1
- net at Q6.4 (G): now also R32.2
- net at Q6.1 (S), Q6.2 (S), Q6.3 (S): now also Q2.1 (S), Q2.2 (S), Q2.3 (S), Q4.1 (S), Q4.2 (S), Q4.3 (S), R33.1, R42.1
- net VCC_3V3: now reaches R9.1
- net VCC_3V3: now also U4.4 (V+)
- net at R9.2: now also C17.1, R3.2, U4.12 (+); no longer Q2.4 (G)
- net at R8.1: now also U3.8 (LO)
- net at R11.1: now also U5.3 (HO)
- new net: C32.1, U5.2 (HB)
- new net: C23.1, U3.2 (HB)
- new net: R7.1, U3.3 (HO)
- new net: R32.1, U5.8 (LO)
- new net: R17.2, R18.2, U4.5 (+)
- new net: Q3.4 (G), R7.2
- new net: Q2.4 (G), R5.2
- new net COMP_CURRENT1: R18.1, U4.13 (-), U4.14
- new net I_SENSE_C: R12.2, U4.7
- new net PWM_B_HS: U3.5 (HI)
- new net PWM_B_LS: U3.6 (LI)
- new net PWM_C_HS: U5.5 (HI)
- new net PWM_C_LS: U5.6 (LI)
- new net V_SENSE_DCBUS: C28.1, R24.2, R25.1
