File: motor1.kicad_sch (KiCad schematic)
At the start: 30 parts, among them Q1 ISCH54N04NM7V, Q2 ISCH54N04NM7V, Q3 ISCH54N04NM7V, Q4 ISCH54N04NM7V, Q5 ISCH54N04NM7V, Q6 ISCH54N04NM7V, U2 UCC27211DRMR, U6 UCC27211DRMR, U7 UCC27211DRMR

Commit message: add
Parts:
- removed C17: 390pF, symbol Device:C_US
- added C17, C31, C35: 0.1uF, symbol Device:C
- added C29, C32, C36, C38, C39: 0.1uF, symbol Device:C_US
- added C30, C33, C34, C37: 2.2uF, symbol Device:C_US
- added R68, R69: 330, symbol Device:R_US
- added R70, R72: 1K, symbol Device:R_US
- added R71, R73: 33K, symbol Device:R_US
- added U14: OPA4376, symbol Amplifier_Operational:OPA4376
- added U18: OPA4374AIPWR, symbol droneUltimate:OPA4374AIPWR
- C18, C19: value 390pF -> 2.2uF
- R10, R14: value 22 -> 68K
- R11, R15: value 22 -> 18K
- R12, R13, R16, R8, R9: value 22 -> 10
- R17: value 4.70K -> 10
- R18, R20: value 1K -> 68K
- R19, R21: value 4.70K -> 18K
- R22: value 1K -> 0.002
- TP2: value HSB -> HSA
- TP3: value HSC -> HSA
Connections:
- net PB_HS_S is gone; now on net BEMF_A: R19.1
- net PC_HS_S is gone; now on an unnamed net: R17.1
- net BEMF_A: now also R10.2, R11.1, R14.2, R15.1, R18.2, C29.1, C32.1, C36.1; no longer C19.1, R21.2, R22.1
- net GNDD: now also R11.2, R15.2, R19.2, R21.2, C29.2, C32.2, C33.2, C36.2, C37.2, C38.2, C39.2, R68.2, R70.1, U14.11 (V-); no longer C18.2, R18.2, R20.2
- net at Q3.1 (S), Q3.2 (S), Q3.3 (S)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: now also R14.1, U6.4 (HS), C31.2
- net at Q3.4 (G): now also R12.2; no longer R11.2
- net VCC_DC+: now reaches Q1.5 (D), Q1.6 (D), Q1.7 (D), Q1.8 (D), Q3.5 (D), Q3.6 (D), Q3.7 (D), Q3.8 (D), Q5.5 (D), Q5.6 (D), Q5.7 (D), Q5.8 (D)
- net VCC_DC+: now also C19.1, R20.1, C33.1, C37.1
- net at Q1.1 (S), Q1.2 (S), Q1.3 (S)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: now also R10.1, U2.4 (HS), C17.2
- net at R12.1: now also U6.3 (HO)
- net VCC: now reaches U2.1 (VDD)
- net VCC: now also C18.1, U6.1 (VDD), U7.1 (VDD), C30.1, C34.1
- net at U2.2 (HB): now also C17.1
- net at U2.3 (HO): now also R8.1
- net PWM_A_HS: now reaches U2.5 (HI)
- net PWM_A_LS: now reaches U2.6 (LI)
- net GNDREF: now reaches U2.7 (VSS)
- net GNDREF: now also C18.2, U2.9 (PAD), U6.7 (VSS), U6.9 (PAD), U7.7 (VSS), U7.9 (PAD), C30.2, C34.2
- net at U2.8 (LO): now also R9.1
- net at Q6.1 (S), Q6.2 (S), Q6.3 (S): now also Q2.1 (S), Q2.2 (S), Q2.3 (S), Q4.1 (S), Q4.2 (S), Q4.3 (S), R22.1, R72.1; no longer R16.2
- net at Q2.4 (G), R9.2: no longer R10.1
- net at U7.2 (HB): now also C35.1
- net at U7.3 (HO): now also R16.1
- net at U7.4 (HS): now also Q5.1 (S), Q5.2 (S), Q5.3 (S), Q6.5 (D), Q6.6 (D), Q6.7 (D), Q6.8 (D), R18.1, TP3.1, C35.2
- net PWM_B_HS: now reaches U7.5 (HI)
- net PWM_B_LS: now reaches U7.6 (LI)
- net at U6.2 (HB): now also C31.1
- net PWM_C_HS: now reaches U6.5 (HI)
- net PWM_C_LS: now reaches U6.6 (LI)
- net at U6.8 (LO): now also R13.1
- net at Q5.4 (G): now also R16.2; no longer R14.2
- removed net BEMF_B: C18.1, R19.2, R20.1
- net BEMF_C: no longer names the net of R17.2
- net BEMF_C: now also Q6.4 (G); no longer R18.1
- net PA_HS_S renamed V_SENSE_DCBUS
- net V_SENSE_DCBUS: now also R20.2, C38.1
- new net: Q4.4 (G), R13.2
- new net: R72.2, R73.1, U18.6 (-)
- new net: R70.2, R71.1, U18.5 (+)
- new net: C39.1, R68.1, R69.2, U18.12 (+)
- new net COMP_CURRENT1: R71.2, U18.13 (-), U18.14
- new net I_SENSE_C: R73.2, U18.7
- new net VCC_3V3: R69.1, U14.4 (V+)
Other:
- moved on the sheet: TP1
