File: motor2.kicad_sch (KiCad schematic)
At the start: 30 parts, among them Q10 ISCH54N04NM7V, Q11 ISCH54N04NM7V, Q12 ISCH54N04NM7V, Q7 ISCH54N04NM7V, Q8 ISCH54N04NM7V, Q9 ISCH54N04NM7V, U3 UCC27211DRMR, U4 UCC27211DRMR, U5 UCC27211DRMR

Commit message: add ti version
Parts:
- removed C22: 390pF, symbol Device:C_US
- removed R23, R24, R25, R30, R31, R32, R35, R36, R37: 22, symbol Device:R_US
- removed R26, R28, R33: 4.70K, symbol Device:R_US
- removed R27: 1K, symbol Device:R_US
- removed U3, U4, U5: UCC27211DRMR, footprints:VSON-8_L4.0-W4.0-P0.80-TL-EP, symbol droneUltimate:UCC27211DRMR
- added C18, C33: 0.1uF, Capacitor_SMD:C_0402_1005Metric, symbol Device:C_US
- added C30, C35, C36, C38, C39, C40: 2.2uF, Capacitor_SMD:C_0402_1005Metric, symbol Device:C_US
- added C42, C43, C52: 0.1uF, Capacitor_SMD:C_0603_1608Metric, symbol Device:C
- added R13: 33K, Resistor_SMD:R_0603_1608Metric, symbol Device:R_US
- added R16: 1K, Resistor_SMD:R_0603_1608Metric, symbol Device:R_US
- added R38, R39, R40, R41, R55, R56: 10, Resistor_SMD:R_0603_1608Metric, symbol Device:R_US
- added R47, R49, R51, R57: 68K, Resistor_SMD:R_0603_1608Metric, symbol Device:R_US
- added R48, R50, R52, R58: 18K, Resistor_SMD:R_0603_1608Metric, symbol Device:R_US
- added R69: 0.002, Resistor_SMD:R_2512_6332Metric, symbol Device:R_US
- added U4: OPA4374AIPWR, footprints:PW14, symbol droneUltimate:OPA4374AIPWR
- added U6, U7, U9: UCC27211DRMR, footprints:VSON-8_L4.0-W4.0-P0.80-TL-EP, symbol droneUltimate:UCC27211DRMR
- C20, C21: value 390pF -> 0.1uF; footprint (none) -> Capacitor_SMD:C_0402_1005Metric; lcsc_id (none) -> C60474; price (none) -> 0.001
- R29: value 1K -> 33K; footprint (none) -> Resistor_SMD:R_0603_1608Metric; lcsc_id (none) -> C2907028; price (none) -> 0.0011
- R34: footprint (none) -> Resistor_SMD:R_0603_1608Metric; lcsc_id (none) -> C2907002; price (none) -> 0.0012
Connections:
- net BEMF_A: now also C20.1, R47.2, R48.1; no longer R34.1
- net BEMF_B: now also R49.2, R50.1; no longer R29.1
- net BEMF_C: now also C18.1, R57.2, R58.1; no longer C20.1
- net GNDD: now also R34.1, C18.2, C33.2, C35.2, C38.2, C40.2, R48.2, R50.2, R52.2, R58.2, R69.2; no longer R29.2, R34.2
- net PA_HS_S: now also Q7.1 (S), Q7.2 (S), Q7.3 (S), Q8.5 (D), Q8.6 (D), Q8.7 (D), Q8.8 (D), TP4.1, C42.2, R47.1, U6.4 (HS)
- net PB_HS_S: now also Q10.5 (D), Q10.6 (D), Q10.7 (D), Q10.8 (D), Q9.1 (S), Q9.2 (S), Q9.3 (S), TP5.1, C43.2, R49.1, U7.4 (HS)
- net PC_HS_S: now also Q11.1 (S), Q11.2 (S), Q11.3 (S), Q12.5 (D), Q12.6 (D), Q12.7 (D), Q12.8 (D), TP6.1, C52.2, R57.1, U9.4 (HS)
- net at Q9.4 (G): now also R55.2
- net at Q8.4 (G): now also R39.2
- net at Q8.1 (S), Q8.2 (S), Q8.3 (S): now also Q10.1 (S), Q10.2 (S), Q10.3 (S), Q12.1 (S), Q12.2 (S), Q12.3 (S), R16.1, R69.1
- net at Q10.4 (G): now also R56.2
- net at Q7.4 (G): now also R38.2
- net VCC_DC+: now reaches Q11.5 (D), Q11.6 (D), Q11.7 (D), Q11.8 (D), Q7.5 (D), Q7.6 (D), Q7.7 (D), Q7.8 (D), Q9.5 (D), Q9.6 (D), Q9.7 (D), Q9.8 (D)
- net VCC_DC+: now also C35.1, C38.1, C40.1, R51.1
- net at Q12.4 (G): now also R41.2
- net at Q11.4 (G): now also R40.2
- new net: C43.1, U7.2 (HB)
- new net: R13.1, R16.2, U4.2 (-)
- new net: R29.2, R34.2, U4.3 (+)
- new net: C42.1, U6.2 (HB)
- new net: R38.1, U6.3 (HO)
- new net: R39.1, U6.8 (LO)
- new net: C52.1, U9.2 (HB)
- new net: R55.1, U7.3 (HO)
- new net: R40.1, U9.3 (HO)
- new net: R41.1, U9.8 (LO)
- new net: R56.1, U7.8 (LO)
- new net COMP_CURRENT1: R29.1
- new net GNDREF: C30.2, C36.2, C39.2, U6.7 (VSS), U6.9 (PAD), U7.7 (VSS), U7.9 (PAD), U9.7 (VSS), U9.9 (PAD)
- new net I_SENSE_C: R13.2, U4.1
- new net PWM_A_HS: U6.5 (HI)
- new net PWM_A_LS: U6.6 (LI)
- new net PWM_B_HS: U7.5 (HI)
- new net PWM_B_LS: U7.6 (LI)
- new net PWM_C_HS: U9.5 (HI)
- new net PWM_C_LS: U9.6 (LI)
- new net VCC_12V: C30.1, C36.1, C39.1, U6.1 (VDD), U7.1 (VDD), U9.1 (VDD)
- new net V_SENSE_DCBUS: C33.1, R51.2, R52.1
