File: motor2.kicad_sch (KiCad schematic)
At the start: 30 parts, among them Q10 ISCH54N04NM7V, Q11 ISCH54N04NM7V, Q12 ISCH54N04NM7V, Q7 ISCH54N04NM7V, Q8 ISCH54N04NM7V, Q9 ISCH54N04NM7V, U3 UCC27211DRMR, U4 UCC27211DRMR, U5 UCC27211DRMR

Commit message: add
Parts:
- removed C21, C22: 390pF, symbol Device:C_US
- removed R23, R24: 22, symbol Device:R_US
- removed U4: UCC27211DRMR, footprints:VSON-8_L4.0-W4.0-P0.80-TL-EP, symbol droneUltimate:UCC27211DRMR
- added C22, C43, C47: 0.1uF, symbol Device:C
- added C40, C42, C44, C46, C50: 2.2uF, symbol Device:C_US
- added C41, C45, C48, C49: 0.1uF, symbol Device:C_US
- added R74, R75: 10, symbol Device:R_US
- added R76, R78: 68K, symbol Device:R_US
- added R77, R79: 18K, symbol Device:R_US
- added U15: UCC27211DRMR, footprints:VSON-8_L4.0-W4.0-P0.80-TL-EP, symbol droneUltimate:UCC27211DRMR
- added U18: OPA4374AIPWR, symbol droneUltimate:OPA4374AIPWR
- C20: value 390pF -> 2.2uF
- R25, R35: value 22 -> 10
- R26: value 4.70K -> 10
- R27: value 1K -> 68K
- R28: value 4.70K -> 18K
- R29: value 1K -> 0.002
- R30, R31: value 22 -> 1K
- R32: value 22 -> 33K
- R33: value 4.70K -> 33K
- R34: value 1K -> 10
- R36: value 22 -> 68K
- R37: value 22 -> 18K
- TP5: value HSB -> HSA
- TP6: value HSC -> HSA
Connections:
- net PB_HS_S is gone; now on net BEMF_A: R28.1
- net PC_HS_S is gone; now on an unnamed net: R26.1
- net BEMF_A: now also R27.2, R36.2, R37.1, C41.1, C45.1, C49.1, R78.2, R79.1; no longer R33.2, R34.1
- net GNDD: now also R28.2, R30.1, R37.2, C41.2, C42.2, C45.2, C46.2, C48.2, C49.2, C50.2, R77.2, R79.2; no longer C20.2, R27.2, R34.2
- net at R30.2: now also R32.1, U18.3 (+); no longer Q9.4 (G)
- net at Q8.4 (G): now also R26.2; no longer R25.1
- net at Q11.1 (S), Q11.2 (S), Q11.3 (S)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: now also C47.2, R78.1, U15.4 (HS)
- net VCC: now reaches U3.1 (VDD)
- net VCC: now also C20.1, U5.1 (VDD), C40.1, C44.1, U15.1 (VDD)
- net at U3.2 (HB): now also C22.1
- net at U3.3 (HO): now also R25.1
- net at U3.4 (HS): now also Q7.1 (S), Q7.2 (S), Q7.3 (S), Q8.5 (D), Q8.6 (D), Q8.7 (D), Q8.8 (D), R27.1, TP4.1, C22.2
- net PWM_A_HS: now reaches U3.5 (HI)
- net PWM_A_LS: now reaches U3.6 (LI)
- net GNDREF: now reaches U3.7 (VSS)
- net GNDREF: now also C20.2, U3.9 (PAD), U5.7 (VSS), U5.9 (PAD), C40.2, C44.2, U15.7 (VSS), U15.9 (PAD)
- net at Q8.1 (S), Q8.2 (S), Q8.3 (S): now also Q10.1 (S), Q10.2 (S), Q10.3 (S), Q12.1 (S), Q12.2 (S), Q12.3 (S), R29.1, R31.1; no longer R25.2
- net at Q10.5 (D), Q10.6 (D), Q10.7 (D)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: now also R36.1, U5.4 (HS), C43.2
- net at Q7.4 (G): now also R25.2
- net VCC_DC+: now reaches Q11.5 (D), Q11.6 (D), Q11.7 (D), Q11.8 (D), Q7.5 (D), Q7.6 (D), Q7.7 (D), Q7.8 (D), Q9.5 (D), Q9.6 (D), Q9.7 (D), Q9.8 (D)
- net VCC_DC+: now also C42.1, C46.1, C50.1, R76.1
- net at R35.2: now also Q10.4 (G); no longer Q11.4 (G)
- net at R35.1: now also U5.8 (LO)
- net at U5.2 (HB): now also C43.1
- net at U5.3 (HO): now also R34.1
- net PWM_C_HS: now reaches U5.5 (HI)
- net PWM_C_LS: now reaches U5.6 (LI)
- removed net BEMF_B: R28.2, R29.1
- removed net BEMF_C: C20.1, R26.2, R27.1
- net PA_HS_S: no longer names the net of R33.1
- net PA_HS_S: now also R31.2, U18.2 (-)
- new net: C47.1, U15.2 (HB)
- new net: R74.1, U15.3 (HO)
- new net: R75.1, U15.8 (LO)
- new net: Q12.4 (G), R75.2
- new net: Q11.4 (G), R74.2
- new net: Q9.4 (G), R34.2
- new net I_SENSE_C: R33.2, U18.1
- new net PWM_B_HS: U15.5 (HI)
- new net PWM_B_LS: U15.6 (LI)
- new net V_SENSE_DCBUS: C48.1, R76.2, R77.1
- now unconnected: R32.2
