File: motor3.kicad_sch (KiCad schematic)
At the start: 30 parts, among them Q13 ISCH54N04NM7V, Q14 ISCH54N04NM7V, Q15 ISCH54N04NM7V, Q16 ISCH54N04NM7V, Q17 ISCH54N04NM7V, Q18 ISCH54N04NM7V, U10 UCC27211DRMR, U8 UCC27211DRMR, U9 UCC27211DRMR

Commit message: add ti version
Parts:
- removed C23, C24, C25: 390pF, symbol Device:C_US
- removed R38, R39, R40, R45, R46, R47, R50, R51, R52: 22, symbol Device:R_US
- removed R41, R48: 4.70K, symbol Device:R_US
- removed R42, R44, R49: 1K, symbol Device:R_US
- removed U8, U9: UCC27211DRMR, footprints:VSON-8_L4.0-W4.0-P0.80-TL-EP, symbol droneUltimate:UCC27211DRMR
- added C41, C44, C45, C50, C56, C59: 2.2uF, Capacitor_SMD:C_0402_1005Metric, symbol Device:C_US
- added C46, C47, C48, C49: 0.1uF, Capacitor_SMD:C_0402_1005Metric, symbol Device:C_US
- added C62, C63, C72: 0.1uF, Capacitor_SMD:C_0603_1608Metric, symbol Device:C
- added R14, R19: 33K, Resistor_SMD:R_0603_1608Metric, symbol Device:R_US
- added R35: 1K, Resistor_SMD:R_0603_1608Metric, symbol Device:R_US
- added R65, R66, R67, R68, R82, R93: 10, Resistor_SMD:R_0603_1608Metric, symbol Device:R_US
- added R74, R76, R78, R84: 68K, Resistor_SMD:R_0603_1608Metric, symbol Device:R_US
- added R75, R77, R79, R85: 18K, Resistor_SMD:R_0603_1608Metric, symbol Device:R_US
- added R91: 0.002, Resistor_SMD:R_2512_6332Metric, symbol Device:R_US
- added U11, U13: UCC27211DRMR, footprints:VSON-8_L4.0-W4.0-P0.80-TL-EP, symbol droneUltimate:UCC27211DRMR
- added U4: OPA4374AIPWR, footprints:PW14, symbol droneUltimate:OPA4374AIPWR
- R43: value 4.70K -> 1K; footprint (none) -> Resistor_SMD:R_0603_1608Metric; lcsc_id (none) -> C2907002; price (none) -> 0.0012
Connections:
- net BEMF_A: now also C47.1, R74.2, R75.1
- net BEMF_B: now also C48.1, R76.2, R77.1; no longer R43.2
- net BEMF_C: now also C46.1, R84.2, R85.1
- net GNDD: now also R43.1, C41.2, C44.2, C45.2, C46.2, C47.2, C48.2, C49.2, R75.2, R77.2, R79.2, R85.2, R91.2
- net PA_HS_S: now also Q13.1 (S), Q13.2 (S), Q13.3 (S), Q14.5 (D), Q14.6 (D), Q14.7 (D), Q14.8 (D), TP7.1, U10.4 (HS), C62.2, R74.1
- net PB_HS_S: now also Q15.1 (S), Q15.2 (S), Q15.3 (S), Q16.5 (D), Q16.6 (D), Q16.7 (D), Q16.8 (D), TP8.1, C63.2, R76.1, U11.4 (HS); no longer R43.1
- net PC_HS_S: now also Q17.1 (S), Q17.2 (S), Q17.3 (S), Q18.5 (D), Q18.6 (D), Q18.7 (D), Q18.8 (D), TP9.1, C72.2, R84.1, U13.4 (HS)
- net at Q14.4 (G): now also R68.2
- net at Q14.1 (S), Q14.2 (S), Q14.3 (S): now also Q16.1 (S), Q16.2 (S), Q16.3 (S), Q18.1 (S), Q18.2 (S), Q18.3 (S), R35.1, R91.1
- net at Q13.4 (G): now also R65.2
- net VCC_DC+: now reaches Q13.5 (D), Q13.6 (D), Q13.7 (D), Q13.8 (D), Q15.5 (D), Q15.6 (D), Q15.7 (D), Q15.8 (D), Q17.5 (D), Q17.6 (D), Q17.7 (D), Q17.8 (D)
- net VCC_DC+: now also C41.1, C44.1, C45.1, R78.1
- net at Q17.4 (G): now also R82.2
- net at Q15.4 (G): now also R67.2
- net at Q18.4 (G): now also R66.2
- net at Q16.4 (G): now also R93.2
- net VCC_12V: now reaches U10.1 (VDD)
- net VCC_12V: now also C50.1, C56.1, C59.1, U11.1 (VDD), U13.1 (VDD)
- net at U10.2 (HB): now also C62.1
- net at U10.3 (HO): now also R65.1
- net PWM_A_HS: now reaches U10.5 (HI)
- net PWM_A_LS: now reaches U10.6 (LI)
- net GNDREF: now reaches U10.7 (VSS)
- net GNDREF: now also U10.9 (PAD), C50.2, C56.2, C59.2, U11.7 (VSS), U11.9 (PAD), U13.7 (VSS), U13.9 (PAD)
- net at U10.8 (LO): now also R68.1
- new net: R14.1, R35.2, U4.9 (-)
- new net: R19.2, R43.2, U4.10 (+)
- new net: R82.1, U13.3 (HO)
- new net: C72.1, U13.2 (HB)
- new net: R66.1, U13.8 (LO)
- new net: R93.1, U11.8 (LO)
- new net: R67.1, U11.3 (HO)
- new net: C63.1, U11.2 (HB)
- new net COMP_CURRENT1: R19.1
- new net I_SENSE_C: R14.2, U4.8
- new net PWM_B_HS: U11.5 (HI)
- new net PWM_B_LS: U11.6 (LI)
- new net PWM_C_HS: U13.5 (HI)
- new net PWM_C_LS: U13.6 (LI)
- new net V_SENSE_DCBUS: C49.1, R78.2, R79.1
