File: motor3.kicad_sch (KiCad schematic)
At the start: 30 parts, among them Q13 ISCH54N04NM7V, Q14 ISCH54N04NM7V, Q15 ISCH54N04NM7V, Q16 ISCH54N04NM7V, Q17 ISCH54N04NM7V, Q18 ISCH54N04NM7V, U10 UCC27211DRMR, U8 UCC27211DRMR, U9 UCC27211DRMR

Commit message: add
Parts:
- removed C24, C25: 390pF, symbol Device:C_US
- removed R38, R39: 22, symbol Device:R_US
- removed U9: UCC27211DRMR, footprints:VSON-8_L4.0-W4.0-P0.80-TL-EP, symbol droneUltimate:UCC27211DRMR
- added C25, C54, C58: 0.1uF, symbol Device:C
- added C51, C53, C55, C57, C61: 2.2uF, symbol Device:C_US
- added C52, C56, C59, C60: 0.1uF, symbol Device:C_US
- added R80, R81: 10, symbol Device:R_US
- added R82, R84: 68K, symbol Device:R_US
- added R83, R85: 18K, symbol Device:R_US
- added U16: UCC27211DRMR, footprints:VSON-8_L4.0-W4.0-P0.80-TL-EP, symbol droneUltimate:UCC27211DRMR
- added U18: OPA4374AIPWR, symbol droneUltimate:OPA4374AIPWR
- added U9: OPA4376, symbol Amplifier_Operational:OPA4376
- C23: value 390pF -> 2.2uF
- R40, R50: value 22 -> 10
- R41: value 4.70K -> 10
- R42: value 1K -> 68K
- R43: value 4.70K -> 18K
- R44: value 1K -> 0.002
- R45, R46: value 22 -> 1K
- R47: value 22 -> 33K
- R48: value 4.70K -> 33K
- R49: value 1K -> 10
- R51: value 22 -> 68K
- R52: value 22 -> 18K
- TP8: value HSB -> HSA
- TP9: value HSC -> HSA
Connections:
- net PB_HS_S is gone; now on net BEMF_A: R43.1
- net PC_HS_S is gone; now on an unnamed net: R41.1
- net BEMF_A: now also R42.2, R51.2, R52.1, C52.1, C56.1, C60.1, R84.2, R85.1; no longer R48.2, R49.1
- net GNDD: now also R43.2, R45.1, R52.2, C52.2, C53.2, C56.2, C57.2, C59.2, C60.2, C61.2, R83.2, R85.2, U9.11 (V-); no longer C23.2, R42.2, R49.2
- net at R40.1: now also U8.3 (HO); no longer Q14.4 (G)
- net at Q14.1 (S), Q14.2 (S), Q14.3 (S): now also Q16.1 (S), Q16.2 (S), Q16.3 (S), Q18.1 (S), Q18.2 (S), Q18.3 (S), R44.1, R46.1; no longer R40.2
- net at Q13.1 (S), Q13.2 (S), Q13.3 (S)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: now also R42.1, U8.4 (HS), C25.2
- net at Q13.4 (G): now also R40.2
- net VCC_DC+: now reaches Q13.5 (D), Q13.6 (D), Q13.7 (D), Q13.8 (D), Q15.5 (D), Q15.6 (D), Q15.7 (D), Q15.8 (D), Q17.5 (D), Q17.6 (D), Q17.7 (D), Q17.8 (D)
- net VCC_DC+: now also C53.1, C57.1, C61.1, R82.1
- net at R50.1: now also U10.8 (LO)
- net at R50.2: now also Q16.4 (G); no longer Q17.4 (G)
- net at R45.2: now also R47.1, U18.10 (+); no longer Q15.4 (G)
- net at Q15.1 (S), Q15.2 (S), Q15.3 (S)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: now also R51.1, U10.4 (HS), C54.2
- net VCC: now reaches U10.1 (VDD)
- net VCC: now also C23.1, U8.1 (VDD), C51.1, C55.1, U16.1 (VDD)
- net at U10.2 (HB): now also C54.1
- net at U10.3 (HO): now also R49.1
- net PWM_C_HS: now reaches U10.5 (HI)
- net PWM_C_LS: now reaches U10.6 (LI)
- net GNDREF: now reaches U10.7 (VSS)
- net GNDREF: now also C23.2, U10.9 (PAD), U8.7 (VSS), U8.9 (PAD), C51.2, C55.2, U16.7 (VSS), U16.9 (PAD)
- net at U8.2 (HB): now also C25.1
- net PWM_A_HS: now reaches U8.5 (HI)
- net PWM_A_LS: now reaches U8.6 (LI)
- net at Q17.1 (S), Q17.2 (S), Q17.3 (S)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: now also C58.2, R84.1, U16.4 (HS)
- removed net BEMF_B: R43.2, R44.1
- removed net BEMF_C: C23.1, R41.2, R42.1
- net PA_HS_S: no longer names the net of R48.1
- net PA_HS_S: now also R46.2, U18.9 (-)
- new net: Q17.4 (G), R80.2
- new net: C58.1, U16.2 (HB)
- new net: R80.1, U16.3 (HO)
- new net: R81.1, U16.8 (LO)
- new net: Q14.4 (G), R41.2
- new net: Q18.4 (G), R81.2
- new net: Q15.4 (G), R49.2
- new net I_SENSE_C: R48.2, U18.8
- new net PWM_B_HS: U16.5 (HI)
- new net PWM_B_LS: U16.6 (LI)
- new net VCC_3V3: U9.4 (V+)
- new net V_SENSE_DCBUS: C59.1, R82.2, R83.1
- now unconnected: R47.2
