File: motor4.kicad_sch (KiCad schematic)
At the start: 30 parts, among them Q19 ISCH54N04NM7V, Q20 ISCH54N04NM7V, Q21 ISCH54N04NM7V, Q22 ISCH54N04NM7V, Q23 ISCH54N04NM7V, Q24 ISCH54N04NM7V, U11 UCC27211DRMR, U12 UCC27211DRMR, U13 UCC27211DRMR

Commit message: add ti version
Parts:
- removed C26, C27, C28: 390pF, symbol Device:C_US
- removed R53, R54, R55, R60, R61, R62, R65, R66, R67: 22, symbol Device:R_US
- removed R56, R58, R63: 4.70K, symbol Device:R_US
- removed R57, R59, R64: 1K, symbol Device:R_US
- removed U11, U12, U13: UCC27211DRMR, footprints:VSON-8_L4.0-W4.0-P0.80-TL-EP, symbol droneUltimate:UCC27211DRMR
- added C25, C58, C60, C70, C76, C79: 2.2uF, Capacitor_SMD:C_0402_1005Metric, symbol Device:C_US
- added C37, C51, C53, C54, C55: 0.1uF, Capacitor_SMD:C_0402_1005Metric, symbol Device:C_US
- added C82, C83, C92: 0.1uF, Capacitor_SMD:C_0603_1608Metric, symbol Device:C
- added R10, R4: 330, Resistor_SMD:R_0402_1005Metric, symbol Device:R_US
- added R100, R28: 33K, Resistor_SMD:R_0603_1608Metric, symbol Device:R_US
- added R101, R103, R105, R111: 68K, Resistor_SMD:R_0603_1608Metric, symbol Device:R_US
- added R102, R104, R106, R112: 18K, Resistor_SMD:R_0603_1608Metric, symbol Device:R_US
- added R109, R86, R87, R88, R89, R92: 10, Resistor_SMD:R_0603_1608Metric, symbol Device:R_US
- added R44, R45: 1K, Resistor_SMD:R_0603_1608Metric, symbol Device:R_US
- added R96: 0.002, Resistor_SMD:R_2512_6332Metric, symbol Device:R_US
- added U14, U15, U17: UCC27211DRMR, footprints:VSON-8_L4.0-W4.0-P0.80-TL-EP, symbol droneUltimate:UCC27211DRMR
- added U16: OPA4374AIPWR, footprints:PW14, symbol droneUltimate:OPA4374AIPWR
Connections:
- net BEMF_A: now also C54.1, R101.2, R102.1
- net BEMF_B: now also C53.1, R103.2, R104.1
- net BEMF_C: now also C55.1, R111.2, R112.1
- net GNDD: now also C25.2, C37.2, C51.2, C53.2, C54.2, C55.2, C58.2, C60.2, R10.1, R102.2, R104.2, R106.2, R112.2, R45.1, R96.2, U16.11 (V-)
- net PA_HS_S: now also Q19.1 (S), Q19.2 (S), Q19.3 (S), Q20.5 (D), Q20.6 (D), Q20.7 (D), Q20.8 (D), TP10.1, C82.2, R101.1, U14.4 (HS)
- net PB_HS_S: now also Q21.1 (S), Q21.2 (S), Q21.3 (S), Q22.5 (D), Q22.6 (D), Q22.7 (D), Q22.8 (D), TP11.1, C83.2, R103.1, U15.4 (HS)
- net PC_HS_S: now also Q23.1 (S), Q23.2 (S), Q23.3 (S), Q24.5 (D), Q24.6 (D), Q24.7 (D), Q24.8 (D), TP12.1, C92.2, R111.1, U17.4 (HS)
- net GNDREF: now reaches Q22.1 (S), Q22.2 (S), Q22.3 (S)
- net GNDREF: now also Q20.1 (S), Q20.2 (S), Q20.3 (S), Q24.1 (S), Q24.2 (S), Q24.3 (S), C70.2, C76.2, C79.2, R44.1, R96.1, U14.7 (VSS), U14.9 (PAD), U15.7 (VSS), U15.9 (PAD), U17.7 (VSS), U17.9 (PAD)
- net at Q22.4 (G): now also R92.2
- net at Q21.4 (G): now also R89.2
- net VCC_DC+: now reaches Q19.5 (D), Q19.6 (D), Q19.7 (D), Q19.8 (D), Q21.5 (D), Q21.6 (D), Q21.7 (D), Q21.8 (D), Q23.5 (D), Q23.6 (D), Q23.7 (D), Q23.8 (D)
- net VCC_DC+: now also C25.1, C58.1, C60.1, R105.1
- net at Q24.4 (G): now also R86.2
- net at Q20.4 (G): now also R88.2
- net at Q23.4 (G): now also R109.2
- net at Q19.4 (G): now also R87.2
- new net: R28.2, R45.2, U16.5 (+)
- new net: R100.1, R44.2, U16.6 (-)
- new net: R86.1, U17.8 (LO)
- new net: R109.1, U17.3 (HO)
- new net: C83.1, U15.2 (HB)
- new net: R89.1, U15.3 (HO)
- new net: R92.1, U15.8 (LO)
- new net: C82.1, U14.2 (HB)
- new net: R88.1, U14.8 (LO)
- new net: C37.1, R10.2, R4.2, U16.12 (+)
- new net: R28.1, U16.13 (-), U16.14
- new net: R87.1, U14.3 (HO)
- new net: C92.1, U17.2 (HB)
- new net I_SENSE_C: R100.2, U16.7
- new net PWM_A_HS: U14.5 (HI)
- new net PWM_A_LS: U14.6 (LI)
- new net PWM_B_HS: U15.5 (HI)
- new net PWM_B_LS: U15.6 (LI)
- new net PWM_C_HS: U17.5 (HI)
- new net PWM_C_LS: U17.6 (LI)
- new net VCC_12V: C70.1, C76.1, C79.1, U14.1 (VDD), U15.1 (VDD), U17.1 (VDD)
- new net VCC_3V3: R4.1, U16.4 (V+)
- new net V_SENSE_DCBUS: C51.1, R105.2, R106.1
