File: motor4.kicad_sch (KiCad schematic)
At the start: 30 parts, among them Q19 ISCH54N04NM7V, Q20 ISCH54N04NM7V, Q21 ISCH54N04NM7V, Q22 ISCH54N04NM7V, Q23 ISCH54N04NM7V, Q24 ISCH54N04NM7V, U11 UCC27211DRMR, U12 UCC27211DRMR, U13 UCC27211DRMR

Commit message: add
Parts:
- removed C28: 390pF, symbol Device:C_US
- removed U12: UCC27211DRMR, footprints:VSON-8_L4.0-W4.0-P0.80-TL-EP, symbol droneUltimate:UCC27211DRMR
- added C28, C65, C69: 0.1uF, symbol Device:C
- added C62, C64, C66, C68, C72: 2.2uF, symbol Device:C_US
- added C63, C67, C70, C71: 0.1uF, symbol Device:C_US
- added R86, R87: 10, symbol Device:R_US
- added R88, R90: 68K, symbol Device:R_US
- added R89, R91: 18K, symbol Device:R_US
- added U12: OPA4376, symbol Amplifier_Operational:OPA4376
- added U17: UCC27211DRMR, footprints:VSON-8_L4.0-W4.0-P0.80-TL-EP, symbol droneUltimate:UCC27211DRMR
- added U4: OPA4374AIPWR, symbol droneUltimate:OPA4374AIPWR
- C26: value 390pF -> 2.2uF
- C27: value 390pF -> 0.1uF
- R53, R54: value 22 -> 330
- R55, R65: value 22 -> 10
- R56: value 4.70K -> 10
- R57: value 1K -> 68K
- R58: value 4.70K -> 18K
- R59: value 1K -> 0.002
- R60, R61: value 22 -> 1K
- R62: value 22 -> 33K
- R63: value 4.70K -> 33K
- R64: value 1K -> 10
- R66: value 22 -> 68K
- R67: value 22 -> 18K
- TP11: value HSB -> HSA
- TP12: value HSC -> HSA
Connections:
- net PB_HS_S is gone; now on net BEMF_A: R58.1
- net PC_HS_S is gone; now on an unnamed net: R56.1
- net BEMF_A: now also R57.2, R66.2, R67.1, C63.1, C67.1, C71.1, R90.2, R91.1; no longer R63.2, R64.1
- net GNDD: now also R54.2, R58.2, R60.1, R67.2, C63.2, C64.2, C67.2, C68.2, C70.2, C71.2, C72.2, R89.2, R91.2, U12.11 (V-); no longer C26.2, R57.2, R64.2
- net at Q21.1 (S), Q21.2 (S), Q21.3 (S)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: now also R66.1, U13.4 (HS), C65.2
- net at Q19.1 (S), Q19.2 (S), Q19.3 (S)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: now also R57.1, U11.4 (HS), C28.2
- net at Q22.1 (S), Q22.2 (S), Q22.3 (S): now also Q20.1 (S), Q20.2 (S), Q20.3 (S), Q24.1 (S), Q24.2 (S), Q24.3 (S), R59.1, R61.1; no longer R62.2
- net at R60.2: now also R62.1, U4.5 (+); no longer Q21.4 (G)
- net VCC_DC+: now reaches Q19.5 (D), Q19.6 (D), Q19.7 (D), Q19.8 (D), Q21.5 (D), Q21.6 (D), Q21.7 (D), Q21.8 (D), Q23.5 (D), Q23.6 (D), Q23.7 (D), Q23.8 (D)
- net VCC_DC+: now also C64.1, C68.1, C72.1, R88.1
- net at Q23.1 (S), Q23.2 (S), Q23.3 (S)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: now also C69.2, R90.1, U17.4 (HS)
- net at R54.1: now also C27.1, R53.2, U4.12 (+)
- net at R65.2: now also Q22.4 (G); no longer Q23.4 (G)
- net at R65.1: now also U13.8 (LO)
- net VCC_3V3: now reaches R53.1
- net VCC_3V3: now also U12.4 (V+)
- net at Q19.4 (G): now also R55.2; no longer R53.2
- net VCC: now reaches U13.1 (VDD)
- net VCC: now also C26.1, U11.1 (VDD), C62.1, C66.1, U17.1 (VDD)
- net at U13.2 (HB): now also C65.1
- net at U13.3 (HO): now also R64.1
- net PWM_C_HS: now reaches U13.5 (HI)
- net PWM_C_LS: now reaches U13.6 (LI)
- net GNDREF: now reaches U13.7 (VSS)
- net GNDREF: now also C26.2, U11.7 (VSS), U11.9 (PAD), U13.9 (PAD), C62.2, C66.2, U17.7 (VSS), U17.9 (PAD)
- net at U11.2 (HB): now also C28.1
- net at U11.3 (HO): now also R55.1
- net PWM_A_HS: now reaches U11.5 (HI)
- net PWM_A_LS: now reaches U11.6 (LI)
- removed net BEMF_B: C27.1, R58.2, R59.1
- removed net BEMF_C: C26.1, R56.2, R57.1
- net PA_HS_S: no longer names the net of R63.1
- net PA_HS_S: now also R61.2, U4.6 (-)
- new net: Q24.4 (G), R87.2
- new net: R87.1, U17.8 (LO)
- new net: Q21.4 (G), R64.2
- new net: C69.1, U17.2 (HB)
- new net: R86.1, U17.3 (HO)
- new net: Q23.4 (G), R86.2
- new net: Q20.4 (G), R56.2
- new net COMP_CURRENT1: R62.2, U4.13 (-), U4.14
- new net I_SENSE_C: R63.2, U4.7
- new net PWM_B_HS: U17.5 (HI)
- new net PWM_B_LS: U17.6 (LI)
- new net V_SENSE_DCBUS: C70.1, R88.2, R89.1
